Commit message: add big car

File: docking_gazebo/urdf/ball.xacro (robot description, xacro)
@@ -4,5 +4,5 @@
     <xacro:macro name="ball" params="fb transX parent">
         <!-- fb: front, back -->
-        <link name="${fb}_ball_link">
+        <link name="${parent}_${fb}_ball_link">
             <visual>
                 <origin xyz="0 0 0 " rpy="0 0 0" />
@@ -20,8 +20,8 @@
             <xacro:sphere_inertial_matrix m="0.01" r="0.04" />
         </link>
-        <gazebo reference="${fb}_ball_link">
+        <gazebo reference="${parent}_${fb}_ball_link">
             <material>Gazebo/Black</material>
         </gazebo>
-        <gazebo reference="${fb}_ball_link">
+        <gazebo reference="${parent}_${fb}_ball_link">
             <mu1>0.01</mu1>
             <mu2>0.01</mu2>
@@ -32,7 +32,7 @@
             <fdir1>0 0 0</fdir1> -->
         </gazebo>
-        <joint name="${fb}_ball_joint" type="fixed">
+        <joint name="${parent}_${fb}_ball_joint" type="fixed">
             <parent link="${parent}"/>
-            <child link="${fb}_ball_link"/>
+            <child link="${parent}_${fb}_ball_link"/>
             <origin xyz="${transX} 0 -0.14" rpy="0 0 0"/>
         </joint>

File: docking_gazebo/urdf/robot.xacro (robot description, xacro)
@@ -2,9 +2,9 @@
 <robot name="robot" xmlns:xacro="http://www.ros.org/wiki/xacro">
     <!-- include -->
-    <xacro:include filename="$(find docking_gazebo)/urdf/inertia.urdf.xacro" />
-    <xacro:include filename="$(find docking_gazebo)/urdf/property.urdf.xacro" />
-    <xacro:include filename="$(find docking_gazebo)/urdf/wheel.urdf.xacro" />
-    <xacro:include filename="$(find docking_gazebo)/urdf/ball.urdf.xacro" />
-    <xacro:include filename="$(find docking_gazebo)/urdf/lidar.urdf.xacro" />
+    <xacro:include filename="$(find docking_gazebo)/urdf/inertia.xacro" />
+    <xacro:include filename="$(find docking_gazebo)/urdf/property.xacro" />
+    <xacro:include filename="$(find docking_gazebo)/urdf/wheel.xacro" />
+    <xacro:include filename="$(find docking_gazebo)/urdf/ball.xacro" />
+    <xacro:include filename="$(find docking_gazebo)/urdf/lidar.xacro" />
     <!-- base_link -->
     <link name="base_link">

File: docking_gazebo/urdf/wheel.xacro (robot description, xacro)
@@ -4,5 +4,5 @@
     <xacro:macro name="wheel" params="lr transY parent">
         <!-- lr: left, right -->
-        <link name="wheel_${lr}_link">
+        <link name="wheel_${parent}_${lr}_link">
             <visual>
                 <origin xyz="0 0 0" rpy="${M_PI/2} 0  0 " />
@@ -20,8 +20,8 @@
             <xacro:cylinder_inertial_matrix m="0.4" r="0.08" h="0.04" />
         </link>
-        <gazebo reference="wheel_${lr}_link">
+        <gazebo reference="wheel_${parent}_${lr}_link">
             <material>Gazebo/Black</material>
         </gazebo>
-        <gazebo reference="wheel_${lr}_link">
+        <gazebo reference="wheel_${parent}_${lr}_link">
             <mu1>5.0</mu1>
             <mu2>1.0</mu2>
@@ -32,7 +32,7 @@
             <fdir1>0 0 0</fdir1>
         </gazebo>
-        <joint name="wheel_${lr}_joint" type="continuous">
+        <joint name="wheel_${parent}_${lr}_joint" type="continuous">
             <parent link="${parent}"/>
-            <child link="wheel_${lr}_link"/>
+            <child link="wheel_${parent}_${lr}_link"/>
             <origin xyz="0 ${transY} -0.1" rpy="0 0 0" />
             <axis xyz="0 1 0" rpy="0 0 0" />

Commit message: modify mass for controlling car
add lidar

File: docking_gazebo/urdf/ball.xacro (robot description, xacro)
@@ -13,10 +13,10 @@
             </visual>
             <collision>
+                <origin xyz="0 0 0 " rpy="0 0 0" />
                 <geometry>
                     <sphere radius="0.04" />
                 </geometry>
-                <origin xyz="0 0 0 " rpy="0 0 0" />
             </collision>
-            <xacro:sphere_inertial_matrix m="0.01" r="0.04" />
+            <xacro:sphere_inertial_matrix m="1e-1" r="0.04" />
         </link>
         <gazebo reference="${parent}_${fb}_ball_link">
@@ -24,6 +24,6 @@
         </gazebo>
         <gazebo reference="${parent}_${fb}_ball_link">
-            <mu1>0.01</mu1>
-            <mu2>0.01</mu2>
+            <mu1>0.001</mu1>
+            <mu2>0.001</mu2>
             <!-- <kp>1000.0</kp>
             <kd>1.0</kd>

File: docking_gazebo/urdf/big_car.xacro (robot description, xacro)
@@ -13,5 +13,5 @@
             </geometry>
         </visual>
-        <xacro:box_inertial_matrix m="1e-4" w="0.93" h="0.1" d="0.1" />
+        <xacro:box_inertial_matrix m="1e-1" w="0.93" h="0.1" d="0.1" />
     </link>
     <gazebo reference="base_link">
@@ -28,24 +28,21 @@
     <gazebo>
         <plugin name="car1_control" filename="libgazebo_ros_diff_drive.so">
-            <rosDebugLevel>Debug</rosDebugLevel>
-            <publishWheelTF>true</publishWheelTF>
-            <robotNamespace>/</robotNamespace>
-            <publishOdomTF>true</publishOdomTF>
-            <publishTf>1</publishTf>
+            <commandTopic>cmd_vel_car1</commandTopic>
+            <odometryTopic>odom_car1</odometryTopic>
+            <odometryFrame>odom</odometryFrame>
+            <robotBaseFrame>big_head</robotBaseFrame>
+            <publishWheelTF>false</publishWheelTF>
             <publishWheelJointState>true</publishWheelJointState>
-            <broadcastTF>1</broadcastTF>
-            <alwaysOn>true</alwaysOn>
-            <updateRate>100.0</updateRate>
             <legacyMode>true</legacyMode>
+            <wheelSeparation>0.37</wheelSeparation>
+            <wheelDiameter>0.16</wheelDiameter>
+            <wheelAcceleration>1.8</wheelAcceleration>
+            <wheelTorque>100</wheelTorque>
+            <updateRate>30.0</updateRate>
             <leftJoint>wheel_car1_left_joint</leftJoint>
             <rightJoint>wheel_car1_right_joint</rightJoint>
-            <wheelSeparation>0.37</wheelSeparation>
-            <wheelDiameter>0.16</wheelDiameter>
-            <wheelTorque>30</wheelTorque>
-            <wheelAcceleration>1.8</wheelAcceleration>
-            <commandTopic>cmd_vel_car1</commandTopic>
-            <odometryFrame>base_link</odometryFrame>
-            <odometryTopic>odom_car1</odometryTopic>
-            <robotBaseFrame>car1</robotBaseFrame>
+            <publishTf>true</publishTf>
+            <rosDebugLevel>na</rosDebugLevel>
+            <publishOdomTF>true</publishOdomTF>
         </plugin>
     </gazebo>
@@ -60,24 +57,21 @@
     <gazebo>
         <plugin name="car2_control" filename="libgazebo_ros_diff_drive.so">
-            <rosDebugLevel>Debug</rosDebugLevel>
-            <publishWheelTF>true</publishWheelTF>
-            <robotNamespace>/</robotNamespace>
-            <publishOdomTF>true</publishOdomTF>
-            <publishTf>1</publishTf>
+            <commandTopic>cmd_vel_car2</commandTopic>
+            <odometryTopic>odom_car2</odometryTopic>
+            <odometryFrame>odom</odometryFrame>
+            <robotBaseFrame>car2</robotBaseFrame>
+            <publishWheelTF>false</publishWheelTF>
             <publishWheelJointState>true</publishWheelJointState>
-            <broadcastTF>1</broadcastTF>
-            <alwaysOn>true</alwaysOn>
-            <updateRate>100.0</updateRate>
             <legacyMode>true</legacyMode>
+            <wheelSeparation>0.37</wheelSeparation>
+            <wheelDiameter>0.16</wheelDiameter>
+            <wheelAcceleration>1.8</wheelAcceleration>
+            <wheelTorque>100</wheelTorque>
+            <updateRate>30.0</updateRate>
             <leftJoint>wheel_car2_left_joint</leftJoint>
             <rightJoint>wheel_car2_right_joint</rightJoint>
-            <wheelSeparation>0.37</wheelSeparation>
-            <wheelDiameter>0.16</wheelDiameter>
-            <wheelTorque>30</wheelTorque>
-            <wheelAcceleration>1.8</wheelAcceleration>
-            <commandTopic>cmd_vel_car2</commandTopic>
-            <odometryFrame>base_link</odometryFrame>
-            <odometryTopic>odom_car2</odometryTopic>
-            <robotBaseFrame>car2</robotBaseFrame>
+            <publishTf>false</publishTf>
+            <rosDebugLevel>na</rosDebugLevel>
+            <publishOdomTF>false</publishOdomTF>
         </plugin>
     </gazebo>

File: docking_gazebo/urdf/lidar.xacro (robot description, xacro)
@@ -1,18 +1,12 @@
 <?xml version="1.0" encoding="utf-8"?>
 <robot xmlns:xacro="http://www.ros.org/wiki/xacro" name="laser">
-    <xacro:macro name="lidar">
-        <joint name="lidar_joint" type="fixed">
-            <parent link="base_link"/>
-            <child link="lidar_link"/>
+    <xacro:macro name="lidar" params="parent">
+        <joint name="${parent}_lidar_joint" type="fixed">
+            <parent link="${parent}"/>
+            <child link="${parent}_lidar_link"/>
             <origin xyz="0.185 0 0.125" rpy="0 0 0" />
         </joint>
-        <link name="lidar_link">
-            <inertial>
-                <mass value="0.1" />
-                <origin xyz="0 0 0" />
-                <inertia ixx="0.01" ixy="0.0" ixz="0.0"
-                         iyy="0.01" iyz="0.0"
-                         izz="0.01" />
-            </inertial>
+        <link name="${parent}_lidar_link">
+            <xacro:cylinder_inertial_matrix m="1e-5" r="0.02" h="0.05" />
             <visual>
                 <origin xyz="0 0 0" rpy="0 0 0" />
@@ -20,5 +14,5 @@
                     <cylinder length="0.05" radius="0.02"/>
                 </geometry>
-                <material name="gray"/>
+                <material name="Black"/>
             </visual>
             <collision>
@@ -29,8 +23,8 @@
             </collision>
         </link>
-        <gazebo reference="lidar_link">
+        <gazebo reference="${parent}_lidar_link">
             <material>Gazebo/Black</material>
         </gazebo>
-        <gazebo reference="lidar_link">
+        <gazebo reference="${parent}_lidar_link">
             <sensor type="ray" name="rplidar">
                 <pose>0 0 0 0 0 0</pose>
@@ -57,7 +51,7 @@
                     </noise>
                 </ray>
-                <plugin name="gazebo_rplidar" filename="libgazebo_ros_laser.so">
-                    <topicName>/scan</topicName>
-                    <frameName>lidar_link</frameName>
+                <plugin name="${parent}_lidar" filename="libgazebo_ros_laser.so">
+                    <topicName>/${parent}_scan</topicName>
+                    <frameName>${parent}_lidar_link</frameName>
                 </plugin>
             </sensor>

File: docking_gazebo/urdf/robot.xacro (robot description, xacro)
@@ -33,5 +33,5 @@
     <xacro:ball fb="back" transX="-0.185" parent="base_link" />
     <!-- Lidar -->
-    <xacro:lidar />
+    <xacro:lidar parent="base_link" />
     <!-- wheel control -->
     <gazebo>

File: docking_gazebo/urdf/small_car.xacro (robot description, xacro)
@@ -2,5 +2,5 @@
 <robot xmlns:xacro="http://www.ros.org/wiki/xacro">
     <xacro:macro name="small_car" params="name">
-        <!-- include -->
+        <!-- # include -->
         <xacro:include filename="$(find docking_gazebo)/urdf/inertia.xacro" />
         <xacro:include filename="$(find docking_gazebo)/urdf/property.xacro" />
@@ -8,5 +8,5 @@
         <xacro:include filename="$(find docking_gazebo)/urdf/ball.xacro" />
         <xacro:include filename="$(find docking_gazebo)/urdf/lidar.xacro" />
-        <!-- base_link -->
+        <!-- # base_link -->
         <link name="${name}">
             <visual>
@@ -22,15 +22,17 @@
                 </geometry>
             </collision>
-            <xacro:box_inertial_matrix m="1.0" w="0.45" h="0.45" d="0.20" />
+            <xacro:box_inertial_matrix m="1e-1" w="0.45" h="0.45" d="0.20" />
         </link>
         <gazebo reference="${name}">
             <material>Gazebo/Blue</material>
         </gazebo>
-        <!-- Wheel Definitions -->
+        <!-- # Wheel Definitions -->
         <xacro:wheel lr="right" transY="0.185" parent="${name}" />
         <xacro:wheel lr="left" transY="-0.185" parent="${name}" />
-        <!-- Ball Definitions -->
+        <!-- # Ball Definitions -->
         <xacro:ball fb="front" transX="0.185" parent="${name}" />
         <xacro:ball fb="back" transX="-0.185" parent="${name}" />
+        <!-- Lidar -->
+        <xacro:lidar parent="${name}" />
     </xacro:macro>
 </robot>

File: docking_gazebo/urdf/wheel.xacro (robot description, xacro)
@@ -18,5 +18,5 @@
                 </geometry>
             </collision>
-            <xacro:cylinder_inertial_matrix m="0.4" r="0.08" h="0.04" />
+            <xacro:cylinder_inertial_matrix m="1e-1" r="0.08" h="0.04" />
         </link>
         <gazebo reference="wheel_${parent}_${lr}_link">

Commit message: replace wheel collision by mesh

File: docking_gazebo/urdf/ball.xacro (robot description, xacro)
@@ -18,5 +18,5 @@
                 </geometry>
             </collision>
-            <xacro:sphere_inertial_matrix m="1e-1" r="0.04" />
+            <xacro:sphere_inertial_matrix m="0.1" r="0.04" />
         </link>
         <gazebo reference="${parent}_${fb}_ball_link">
@@ -24,11 +24,6 @@
         </gazebo>
         <gazebo reference="${parent}_${fb}_ball_link">
-            <mu1>0.001</mu1>
-            <mu2>0.001</mu2>
-            <!-- <kp>1000.0</kp>
-            <kd>1.0</kd>
-            <minDepth>0.0</minDepth>
-            <maxVel>5</maxVel>
-            <fdir1>0 0 0</fdir1> -->
+            <mu1>0.0001</mu1>
+            <mu2>0.0001</mu2>
         </gazebo>
         <joint name="${parent}_${fb}_ball_joint" type="fixed">

File: docking_gazebo/urdf/big_car.xacro (robot description, xacro)
@@ -36,7 +36,7 @@
             <legacyMode>true</legacyMode>
             <wheelSeparation>0.37</wheelSeparation>
-            <wheelDiameter>0.16</wheelDiameter>
+            <wheelDiameter>0.066</wheelDiameter>
             <wheelAcceleration>1.8</wheelAcceleration>
-            <wheelTorque>100</wheelTorque>
+            <wheelTorque>10</wheelTorque>
             <updateRate>30.0</updateRate>
             <leftJoint>wheel_car1_left_joint</leftJoint>
@@ -65,7 +65,7 @@
             <legacyMode>true</legacyMode>
             <wheelSeparation>0.37</wheelSeparation>
-            <wheelDiameter>0.16</wheelDiameter>
+            <wheelDiameter>0.066</wheelDiameter>
             <wheelAcceleration>1.8</wheelAcceleration>
-            <wheelTorque>100</wheelTorque>
+            <wheelTorque>10</wheelTorque>
             <updateRate>30.0</updateRate>
             <leftJoint>wheel_car2_left_joint</leftJoint>

File: docking_gazebo/urdf/small_car.xacro (robot description, xacro)
@@ -23,5 +23,5 @@
                 </geometry>
             </collision>
-            <xacro:box_inertial_matrix m="1.0" w="0.45" h="0.45" d="0.20" />
+            <xacro:box_inertial_matrix m="10.0" w="0.45" h="0.45" d="0.20" />
         </link>
         <gazebo reference="${name}">

File: docking_gazebo/urdf/wheel.xacro (robot description, xacro)
@@ -4,38 +4,37 @@
     <xacro:macro name="wheel" params="lr transY parent">
         <!-- lr: left, right -->
-        <link name="wheel_${parent}_${lr}_link">
-            <visual>
-                <origin xyz="0 0 0" rpy="${M_PI/2} 0  0 " />
-                <geometry>
-                    <cylinder length="0.04" radius="0.08" />
-                </geometry>
-                <material name="Black" />
-            </visual>
-            <collision>
-                <origin xyz="0 0 0" rpy="${M_PI/2} 0 0 " />
-                <geometry>
-                    <cylinder length="0.04" radius="0.08" />
-                </geometry>
-            </collision>
-            <xacro:cylinder_inertial_matrix m="1e-1" r="0.08" h="0.04" />
-        </link>
         <gazebo reference="wheel_${parent}_${lr}_link">
             <material>Gazebo/Black</material>
         </gazebo>
         <gazebo reference="wheel_${parent}_${lr}_link">
-            <mu1>5.0</mu1>
+            <mu1>10.0</mu1>
             <mu2>1.0</mu2>
             <kp>10000.0</kp>
-            <kd>10.0</kd>
+            <kd>1.0</kd>
             <minDepth>0.0</minDepth>
-            <maxVel>5</maxVel>
-            <fdir1>0 0 0</fdir1>
+            <maxVel>100</maxVel>
+            <fdir1>1 0 0</fdir1>
         </gazebo>
         <joint name="wheel_${parent}_${lr}_joint" type="continuous">
             <parent link="${parent}"/>
             <child link="wheel_${parent}_${lr}_link"/>
-            <origin xyz="0 ${transY} -0.1" rpy="0 0 0" />
+            <origin xyz="0 ${transY} -0.15" rpy="0 0 0" />
             <axis xyz="0 1 0" rpy="0 0 0" />
         </joint>
+        <link name="wheel_${parent}_${lr}_link">
+            <visual>
+                <origin xyz="0 0 0" rpy="0 0 0"/>
+                <geometry>
+                    <mesh filename="package://docking_gazebo/mesh/right_tire.stl" scale="0.001 0.001 0.001"/>
+                </geometry>
+            </visual>
+            <collision>
+                <origin xyz="0 0 0" rpy="0 0 0"/>
+                <geometry>
+                    <mesh filename="package://docking_gazebo/mesh/right_tire.stl" scale="0.001 0.001 0.001"/>
+                </geometry>
+            </collision>
+            <xacro:cylinder_inertial_matrix m="1.0" r="0.08" h="0.04" />
+        </link>
     </xacro:macro>
 </robot>
