Commit message: rm submodule move_base

File: docking_gazebo/urdf/lidar.xacro (robot description, xacro)
@@ -5,5 +5,5 @@
             <parent link="${parent}"/>
             <child link="${parent}_lidar_link"/>
-            <origin xyz="0 0 0.125" rpy="0 0 0" />
+            <origin xyz="0.1 0 0.125" rpy="0 0 0" />
         </joint>
         <link name="${parent}_lidar_link">
