Commit message: car2

File: docking_gazebo/urdf/big_car.xacro (robot description, xacro)
@@ -10,8 +10,8 @@
             <origin xyz="-0.465 0 0.3" rpy="0 0 0" />
             <geometry>
-                <box size="0.93 0.1 0.1" />
+                <box size="0.93 0.1 0.05" />
             </geometry>
         </visual>
-        <xacro:box_inertial_matrix m="0.01" w="0.93" h="0.1" d="0.1" />
+        <xacro:box_inertial_matrix m="1e-4" w="0.93" h="0.1" d="0.1" />
     </link>
     <gazebo reference="base_link">
@@ -20,9 +20,8 @@
     <!-- # small car 1 -->
     <xacro:small_car name="car1" />
-    <joint name="car1_joint" type="fixed">
-    <!-- <joint name="car1_joint" type="continuous"> -->
-        <parent link="base_link"/>
-        <child link="car1"/>
-        <origin xyz="0.0 0.0 0.0" rpy="0 0 0" />
+    <joint name="car1_joint" type="continuous">
+        <parent link="base_link" />
+        <child link="car1" />
+        <origin xyz="0 0 0" rpy="0 0 0" />
         <axis xyz="0 0 1" rpy="0 0 0" />
     </joint>
@@ -46,5 +45,5 @@
             <wheelAcceleration>1.8</wheelAcceleration>
             <commandTopic>cmd_vel_car1</commandTopic>
-            <odometryFrame>odom</odometryFrame>
+            <odometryFrame>base_link</odometryFrame>
             <odometryTopic>odom_car1</odometryTopic>
             <robotBaseFrame>car1</robotBaseFrame>
@@ -52,12 +51,12 @@
     </gazebo>
     <!-- # small car 2 -->
-    <!-- <xacro:small_car name="car2" />
-    <joint name="car2_joint" type="fixed">
-        <parent link="base_link"/>
-        <child link="car2"/>
-        <origin xyz="-0.93 0.0 0.0" rpy="0 0 0" />
+    <xacro:small_car name="car2" />
+    <joint name="car2_joint" type="continuous">
+        <parent link="base_link" />
+        <child link="car2" />
+        <origin xyz="-0.93 0 0" rpy="0 0 0" />
         <axis xyz="0 0 1" rpy="0 0 0" />
-    </joint> -->
-    <!-- <gazebo>
+    </joint>
+    <gazebo>
         <plugin name="car2_control" filename="libgazebo_ros_diff_drive.so">
             <rosDebugLevel>Debug</rosDebugLevel>
@@ -78,8 +77,8 @@
             <wheelAcceleration>1.8</wheelAcceleration>
             <commandTopic>cmd_vel_car2</commandTopic>
-            <odometryFrame>odom</odometryFrame>
+            <odometryFrame>base_link</odometryFrame>
             <odometryTopic>odom_car2</odometryTopic>
             <robotBaseFrame>car2</robotBaseFrame>
         </plugin>
-    </gazebo> -->
+    </gazebo>
 </robot>

File: docking_gazebo/urdf/small_car.xacro (robot description, xacro)
@@ -22,5 +22,5 @@
                 </geometry>
             </collision>
-            <xacro:box_inertial_matrix m="10.0" w="0.45" h="0.45" d="0.20" />
+            <xacro:box_inertial_matrix m="1.0" w="0.45" h="0.45" d="0.20" />
         </link>
         <gazebo reference="${name}">

Commit message: add big_car_tf_br.py

File: docking_gazebo/urdf/big_car.xacro (robot description, xacro)
@@ -8,10 +8,10 @@
     <link name="base_link">
         <visual>
-            <origin xyz="-0.465 0 0.3" rpy="0 0 0" />
+            <origin xyz="0 0 0.3" rpy="0 0 0" />
             <geometry>
                 <box size="0.93 0.1 0.05" />
             </geometry>
         </visual>
-        <xacro:box_inertial_matrix m="1e-1" w="0.93" h="0.1" d="0.1" />
+        <xacro:box_inertial_matrix m="1e-1" w="0.93" h="0.1" d="0.05" />
     </link>
     <gazebo reference="base_link">
@@ -23,5 +23,5 @@
         <parent link="base_link" />
         <child link="car1" />
-        <origin xyz="0 0 0" rpy="0 0 0" />
+        <origin xyz="0.465 0 0" rpy="0 0 0" />
         <axis xyz="0 0 1" rpy="0 0 0" />
     </joint>
@@ -31,5 +31,5 @@
             <odometryTopic>odom_car1</odometryTopic>
             <odometryFrame>odom</odometryFrame>
-            <robotBaseFrame>big_head</robotBaseFrame>
+            <robotBaseFrame>base_link</robotBaseFrame>
             <publishWheelTF>false</publishWheelTF>
             <publishWheelJointState>true</publishWheelJointState>
@@ -52,5 +52,5 @@
         <parent link="base_link" />
         <child link="car2" />
-        <origin xyz="-0.93 0 0" rpy="0 0 0" />
+        <origin xyz="-0.465 0 0" rpy="0 0 0" />
         <axis xyz="0 0 1" rpy="0 0 0" />
     </joint>
@@ -60,5 +60,5 @@
             <odometryTopic>odom_car2</odometryTopic>
             <odometryFrame>odom</odometryFrame>
-            <robotBaseFrame>car2</robotBaseFrame>
+            <robotBaseFrame>base_link</robotBaseFrame>
             <publishWheelTF>false</publishWheelTF>
             <publishWheelJointState>true</publishWheelJointState>

File: docking_gazebo/urdf/imu.xacro (robot description, xacro)
@@ -2,6 +2,11 @@
 <robot xmlns:xacro="http://www.ros.org/wiki/xacro">
     <xacro:macro name="imu" params="parent">
+        <joint name="${parent}_imu_joint" type="fixed">
+            <parent link="${parent}"/>
+            <child link="${parent}_imu_link"/>
+            <origin xyz="0 0 0.12" rpy="0 0 0" />
+        </joint>
         <link name="${parent}_imu_link">
-            <xacro:cylinder_inertial_matrix m="1e-5" r="0.02" h="0.05" />
+            <xacro:cylinder_inertial_matrix m="1e-5" r="0.01" h="0.01" />
             <visual>
                 <origin xyz="0 0 0" rpy="0 0 0" />
@@ -22,5 +27,5 @@
                 <topic>__default_topic__</topic>
                 <plugin filename="libgazebo_ros_imu_sensor.so" name="${parent}_imu_plugin">
-                <topicName>imu</topicName>
+                <topicName>${parent}_imu</topicName>
                 <bodyName>${parent}_imu_link</bodyName>
                 <updateRateHZ>10.0</updateRateHZ>

File: docking_gazebo/urdf/lidar.xacro (robot description, xacro)
@@ -14,12 +14,5 @@
                     <cylinder length="0.05" radius="0.02"/>
                 </geometry>
-                <material name="Black"/>
             </visual>
-            <collision>
-                <origin xyz="0 0 0" rpy="0 0 0" />
-                <geometry>
-                    <cylinder length="0.01" radius="0.01"/>
-                </geometry>
-            </collision>
         </link>
         <gazebo reference="${parent}_lidar_link">

File: docking_gazebo/urdf/small_car.xacro (robot description, xacro)
@@ -8,4 +8,5 @@
         <xacro:include filename="$(find docking_gazebo)/urdf/ball.xacro" />
         <xacro:include filename="$(find docking_gazebo)/urdf/lidar.xacro" />
+        <xacro:include filename="$(find docking_gazebo)/urdf/imu.xacro" />
         <!-- # base_link -->
         <link name="${name}">
@@ -35,4 +36,6 @@
         <!-- Lidar -->
         <xacro:lidar parent="${name}" />
+        <!-- IMU -->
+        <xacro:imu parent="${name}" />
     </xacro:macro>
 </robot>

Commit message: debug orientation error

File: docking_gazebo/urdf/big_car.xacro (robot description, xacro)
@@ -13,5 +13,5 @@
             </geometry>
         </visual>
-        <xacro:box_inertial_matrix m="1e-1" w="0.93" h="0.1" d="0.05" />
+        <xacro:box_inertial_matrix m="1e-2" w="0.93" h="0.1" d="0.05" />
     </link>
     <gazebo reference="base_link">

File: docking_gazebo/urdf/imu.xacro (robot description, xacro)
@@ -5,5 +5,5 @@
             <parent link="${parent}"/>
             <child link="${parent}_imu_link"/>
-            <origin xyz="0 0 0.12" rpy="0 0 0" />
+            <origin xyz="0 0 0.2" rpy="0 0 0" />
         </joint>
         <link name="${parent}_imu_link">

File: docking_gazebo/urdf/inertia.xacro (robot description, xacro)
@@ -6,6 +6,6 @@
             <mass value="${m}" />
             <inertia ixx="${2*m*r*r/5}" ixy="0" ixz="0"
-                iyy="${2*m*r*r/5}" iyz="0"
-                izz="${2*m*r*r/5}" />
+                     iyy="${2*m*r*r/5}" iyz="0"
+                     izz="${2*m*r*r/5}" />
         </inertial>
     </xacro:macro>
@@ -14,6 +14,6 @@
             <mass value="${m}" />
             <inertia ixx="${m*(3*r*r+h*h)/12}" ixy = "0" ixz = "0"
-                iyy="${m*(3*r*r+h*h)/12}" iyz = "0"
-                izz="${m*r*r/2}" />
+                     iyy="${m*(3*r*r+h*h)/12}" iyz = "0"
+                     izz="${m*r*r/2}" />
         </inertial>
     </xacro:macro>
@@ -22,6 +22,6 @@
             <mass value="${m}" />
             <inertia ixx="${m*(h*h+d*d)/12}" ixy = "0" ixz = "0"
-                iyy="${m*(w*w+d*d)/12}" iyz = "0"
-                izz="${m*(w*w+h*h)/12}" />
+                     iyy="${m*(w*w+d*d)/12}" iyz = "0"
+                     izz="${m*(w*w+h*h)/12}" />
         </inertial>
     </xacro:macro>

File: docking_gazebo/urdf/lidar.xacro (robot description, xacro)
@@ -5,5 +5,5 @@
             <parent link="${parent}"/>
             <child link="${parent}_lidar_link"/>
-            <origin xyz="0.185 0 0.125" rpy="0 0 0" />
+            <origin xyz="0 0 0.125" rpy="0 0 0" />
         </joint>
         <link name="${parent}_lidar_link">

File: docking_gazebo/urdf/small_car.xacro (robot description, xacro)
@@ -23,5 +23,5 @@
                 </geometry>
             </collision>
-            <xacro:box_inertial_matrix m="1e-1" w="0.45" h="0.45" d="0.20" />
+            <xacro:box_inertial_matrix m="1.0" w="0.45" h="0.45" d="0.20" />
         </link>
         <gazebo reference="${name}">

Commit message: make follower face backward initially

File: docking_gazebo/urdf/big_car.xacro (robot description, xacro)
@@ -19,5 +19,5 @@
     </gazebo>
     <!-- # small car 1 -->
-    <xacro:small_car name="car1" />
+    <xacro:small_car name="car1" yaw_offset="0" />
     <joint name="car1_joint" type="continuous">
         <parent link="base_link" />
@@ -48,9 +48,9 @@
     </gazebo>
     <!-- # small car 2 -->
-    <xacro:small_car name="car2" />
+    <xacro:small_car name="car2" yaw_offset="3.14" />
     <joint name="car2_joint" type="continuous">
         <parent link="base_link" />
         <child link="car2" />
-        <origin xyz="-0.465 0 0" rpy="0 0 0" />
+        <origin xyz="-0.465 0 0" rpy="0 0 3.14" />
         <axis xyz="0 0 1" rpy="0 0 0" />
     </joint>

File: docking_gazebo/urdf/imu.xacro (robot description, xacro)
@@ -1,5 +1,5 @@
 <?xml version="1.0" encoding="utf-8"?>
 <robot xmlns:xacro="http://www.ros.org/wiki/xacro">
-    <xacro:macro name="imu" params="parent">
+    <xacro:macro name="imu" params="parent yaw_offset">
         <joint name="${parent}_imu_joint" type="fixed">
             <parent link="${parent}"/>
@@ -32,5 +32,5 @@
                 <gaussianNoise>0.0</gaussianNoise>
                 <xyzOffset>0 0 0</xyzOffset>
-                <rpyOffset>0 0 0</rpyOffset>
+                <rpyOffset>0 0 ${yaw_offset}</rpyOffset>
                 <frameName>${parent}_imu_link</frameName>
             </plugin>

File: docking_gazebo/urdf/small_car.xacro (robot description, xacro)
@@ -1,5 +1,5 @@
 <?xml version="1.0" encoding="utf-8"?>
 <robot xmlns:xacro="http://www.ros.org/wiki/xacro">
-    <xacro:macro name="small_car" params="name">
+    <xacro:macro name="small_car" params="name yaw_offset">
         <!-- # include -->
         <xacro:include filename="$(find docking_gazebo)/urdf/inertia.xacro" />
@@ -37,5 +37,5 @@
         <xacro:lidar parent="${name}" />
         <!-- IMU -->
-        <xacro:imu parent="${name}" />
+        <xacro:imu parent="${name}" yaw_offset="${yaw_offset}"/>
     </xacro:macro>
 </robot>

Commit message: add double shelf stl

File: docking_gazebo/urdf/big_car.xacro (robot description, xacro)
@@ -8,7 +8,12 @@
     <link name="base_link">
         <visual>
-            <origin xyz="0 0 0.3" rpy="0 0 0" />
+            <!-- <origin xyz="0 0 0.3" rpy="0 0 0" />
             <geometry>
                 <box size="0.93 0.1 0.05" />
+            </geometry> -->
+            <origin xyz="0 0 0.36" rpy="0 0 0" />
+            <transparency>1</transparency>
+            <geometry>
+                <mesh filename="package://docking_gazebo/mesh/double_shelf_v2.stl" />
             </geometry>
         </visual>
@@ -16,5 +21,5 @@
     </link>
     <gazebo reference="base_link">
-        <material>Gazebo/Blue</material>
+        <material>Gazebo/Gray</material>
     </gazebo>
     <!-- # small car 1 -->

Commit message: add shelf collision for lidar

File: docking_gazebo/urdf/big_car.xacro (robot description, xacro)
@@ -10,13 +10,18 @@
             <!-- <origin xyz="0 0 0.3" rpy="0 0 0" />
             <geometry>
-                <box size="0.93 0.1 0.05" />
+                <box size="1.0 0.1 0.05" />
             </geometry> -->
-            <origin xyz="0 0 0.36" rpy="0 0 0" />
-            <transparency>1</transparency>
+            <origin xyz="0 0 0.38" rpy="0 0 0" />
             <geometry>
                 <mesh filename="package://docking_gazebo/mesh/double_shelf_v2.stl" />
             </geometry>
         </visual>
-        <xacro:box_inertial_matrix m="1.0" w="0.93" h="0.1" d="0.05" />
+        <collision>
+            <origin xyz="0 0 0.38" rpy="0 0 0" />
+            <geometry>
+                <mesh filename="package://docking_gazebo/mesh/double_shelf_v2.stl" />
+            </geometry>
+        </collision>
+        <xacro:box_inertial_matrix m="1.0" w="1.0" h="0.1" d="0.05" />
     </link>
     <gazebo reference="base_link">
@@ -28,5 +33,5 @@
         <parent link="base_link" />
         <child link="car1" />
-        <origin xyz="0.465 0 0" rpy="0 0 0" />
+        <origin xyz="0.5 0 0" rpy="0 0 0" />
         <axis xyz="0 0 1" rpy="0 0 0" />
     </joint>
@@ -57,5 +62,6 @@
         <parent link="base_link" />
         <child link="car2" />
-        <origin xyz="-0.465 0 0" rpy="0 0 3.14" />
+        <!-- <origin xyz="-0.465 0 0" rpy="0 0 3.14" /> -->
+        <origin xyz="-0.5 0 0" rpy="0 0 3.14" />
         <axis xyz="0 0 1" rpy="0 0 0" />
     </joint>
